File: Electronics and Wiring/Wiring.sch (EAGLE design)
At the start: 46 parts, among them K1 SSR-10A-ZERO-CROSS, K2 SSR-10A-ZERO-CROSS, SW1 CT10-XXXX-A2

Commit message: Updating the wiring schematic.
Parts:
- removed U$4: MALE-SOCKET, Edited Parts:MALE-SOCKET
- added GFCI-INLINE: GFCI-INLINE, Edited Parts:GFCI-INLINE
- added MALE-SOCKET: MALE-SOCKET, Edited Parts:MALE-SOCKET
- added WATERBATH-CHASSIS: Ring terminal and screw, SparkFun-Connectors:CONN_01
Connections:
- new net N$74: GFCI-INLINE.L-OUT, MALE-SOCKET.L-IN
- new net N$75: GFCI-INLINE.N-OUT, MALE-SOCKET.N-IN
- new net N$76: GFCI-INLINE.G-OUT, MALE-SOCKET.G-IN
- new net N$77: GFCI-INLINE.L-IN
- new net N$78: GFCI-INLINE.N-IN
- new net N$79: GFCI-INLINE.G-IN
- net N$1: now also MALE-SOCKET.L-OUT; no longer U$4.L-OUT
- net N$4: now also MALE-SOCKET.N-OUT; no longer U$4.N-OUT
- net N$5: now also MALE-SOCKET.G-OUT, WATERBATH-CHASSIS.1; no longer U$4.G-OUT
- net N$67: now also U$3.KPD-2
- net N$69: now also U$3.KPD-4
- net N$70: now also U$3.KPD-5
Other:
- note added: "Extruder Body and Gear Box"
- note added: "Low Voltage Electronics"
- note added: "Mains Power"
- note added: "Mains Voltage Electronics"
- note added: "Power cord"
- note added: "Thunderhead Filament Extrtuder Overall Wiring Diagram"
- note added: "Waterbath and Outfeed"
- moved on the sheet: K1, K2, PRIMARY-NC-DIA-SENSOR, QC-NC-DIA-SENSOR, U$2, U$3, WIRENUT-10, WIRENUT-11, WIRENUT-12, WIRENUT-13, WIRENUT-14, WIRENUT-15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

Commit message: Updating electronics files
Parts:
- removed WIRENUT-19, WIRENUT-20, WIRENUT-21: (no value), SparkFun-Connectors:CONN_01
- added HEADER-OR-WIRENUT-2, HEADER-OR-WIRENUT-3, HEADER-OR-WIRENUT-4: (no value), SparkFun-Connectors:CONN_01
- renumbered WIRENUT-18 to HEADER-OR-WIRENUT-1
Connections:
- net N$3: now also U$3.12V-Z345
- net N$47: now also HEADER-OR-WIRENUT-2.1; no longer WIRENUT-19.1
- net N$48: now also HEADER-OR-WIRENUT-3.1; no longer WIRENUT-20.1
- net N$49: now also HEADER-OR-WIRENUT-4.1; no longer WIRENUT-21.1
- net N$6: now also U$3.GND-Z345
