File: Electronics and Wiring/Thunderboard.sch (EAGLE design)
At the start: 33 parts, among them Q1 TIP120, Q2 TIP120, Q3 TIP120, T1 2n2222

Commit message: Updating electronics files
Parts:
- R9: value 1K -> 3K
- T1: value 2n2222 -> PN2222A
Changed lines of the file:
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@@
 <part name="Q3" library="Edited Parts" deviceset="TIP120" device="" package3d_urn="urn:adsk.eagle:package:29488/1"/>
 <part name="5V-PIEZO-BUZZER" library="SparkFun-Electromechanical" deviceset="BUZZER" device="-PTH"/>
-<part name="T1" library="transistor" library_urn="urn:adsk.eagle:library:402" deviceset="*-NPN-" device="TO92-EBC" package3d_urn="urn:adsk.eagle:package:29915/2" value="2n2222"/>
-<part name="R9" library="resistor - edit" deviceset="R-US_" device="0207/7" package3d_urn="urn:adsk.eagle:package:25942/1" value="1K"/>
+<part name="T1" library="transistor" library_urn="urn:adsk.eagle:library:402" deviceset="*-NPN-" device="TO92-EBC" package3d_urn="urn:adsk.eagle:package:29915/2" value="PN2222A"/>
+<part name="R9" library="resistor - edit" deviceset="R-US_" device="0207/7" package3d_urn="urn:adsk.eagle:package:25942/1" value="3K"/>
 <part name="IIC-1" library="SparkFun-Connectors" library_urn="urn:adsk.eagle:library:513" deviceset="CONN_04" device="" package3d_urn="urn:adsk.eagle:package:38085/1"/>
 <part name="IIC-2" library="SparkFun-Connectors" library_urn="urn:adsk.eagle:library:513" deviceset="CONN_04" device="" package3d_urn="urn:adsk.eagle:package:38085/1"/>

Commit message: Changes made after testing the Thunderboard. Switched from Tip120 to a power fet STP55NF06L.
Parts:
- added R11, R12, R13: 100k, resistor - edit:R-US_0207/7
- F1: value (none) -> 10 A
- F2: value (none) -> 5A
- Q1, Q2, Q3: value TIP120 -> STP55NF06L; device Edited Parts:TIP120 -> Edited Parts:STP55NF06L
- R6, R7, R8: value 1K -> 100R
Connections:
- net D10: now also R11.1
- net D8: now also R13.1
- net D9: now also R12.1
- net GND: now also Q1.S, Q2.S, Q3.S, R11.2, R12.2, R13.2; no longer Q1.E, Q2.E, Q3.E
- net N$10: now also Q3.D; no longer Q3.C
- net N$3: now also Q1.G; no longer Q1.B
- net N$4: now also Q2.G; no longer Q2.B
- net N$5: now also Q3.G; no longer Q3.B
- net N$7: now also Q1.D; no longer Q1.C
- net N$9: now also Q2.D; no longer Q2.C
Other:
- moved on the sheet: R6, R7, R8, Z3, Z4, Z5
